Commit message: [feat]:给夹爪添加位控制器

File: src/arm_description/urdf/robot.ros_control.xacro (robot description, xacro)
@@ -34,4 +34,44 @@
             </actuator>
         </transmission>
+        <transmission name="finger1_transmission">
+            <type>transmission_interface/SimpleTransmission</type>
+            <joint name="finger1_joint">
+                <hardwareInterface>hardware_interface/PositionJointInterface</hardwareInterface>
+            </joint>
+            <actuator name="finger1_motor">
+                <hardwareInterface>hardware_interface/PositionJointInterface</hardwareInterface>
+                <mechanicalReduction>1</mechanicalReduction>
+            </actuator>
+        </transmission>
+        <transmission name="finger2_transmission">
+            <type>transmission_interface/SimpleTransmission</type>
+            <joint name="finger2_joint">
+                <hardwareInterface>hardware_interface/PositionJointInterface</hardwareInterface>
+            </joint>
+            <actuator name="finger2_motor">
+                <hardwareInterface>hardware_interface/PositionJointInterface</hardwareInterface>
+                <mechanicalReduction>1</mechanicalReduction>
+            </actuator>
+        </transmission>
+        <transmission name="finger3_transmission">
+            <type>transmission_interface/SimpleTransmission</type>
+            <joint name="finger3_joint">
+                <hardwareInterface>hardware_interface/PositionJointInterface</hardwareInterface>
+            </joint>
+            <actuator name="finger3_motor">
+                <hardwareInterface>hardware_interface/PositionJointInterface</hardwareInterface>
+                <mechanicalReduction>1</mechanicalReduction>
+            </actuator>
+        </transmission>
+        <transmission name="finger4_transmission">
+            <type>transmission_interface/SimpleTransmission</type>
+            <joint name="finger4_joint">
+                <hardwareInterface>hardware_interface/PositionJointInterface</hardwareInterface>
+            </joint>
+            <actuator name="finger4_motor">
+                <hardwareInterface>hardware_interface/PositionJointInterface</hardwareInterface>
+                <mechanicalReduction>1</mechanicalReduction>
+            </actuator>
+        </transmission>
         <!-- Gazebo ros_control plugin -->
         <gazebo>
