Commit message: [fix]:改变urdf限位,成功实现坐标转换\夹取,至此,pybullet上完成的工作已在gazebo上复现.下一步是规范化夹取流程,主要从以下几点考虑:1. 夹取动作规划,先移到上方,再下降机械臂;2. 下降高度根据物体高度自动确定

File: src/arm_description/urdf/base.urdf.xacro (robot description, xacro)
@@ -37,5 +37,5 @@
             <origin xyz="0 0 0.4" rpy="0 0 0"/>
             <axis xyz="0 0 1"/>
-            <limit effort="20" velocity="2.0" lower="-2.6" upper="2.6"/>
+            <limit effort="20" velocity="2.0" lower="-3.2" upper="3.2"/>
             <dynamics damping="0.1" friction="0.05"/>
         </joint>
@@ -70,5 +70,5 @@
             <origin xyz="0 -1.0 0.1" rpy="0 0 0"/>
             <axis xyz="0 0 1"/>
-            <limit effort="15" velocity="2.0" lower="-3.00" upper="3.00"/>
+            <limit effort="15" velocity="2.0" lower="-3.2" upper="3.2"/>
             <dynamics damping="0.1" friction="0.05"/>
         </joint>

Commit message: [feat]：增大手指面积，部分解决夹爪夹不起来的问题，但目前会有穿模问题，考虑再加一个旋转关节

File: src/arm_description/urdf/base.urdf.xacro (robot description, xacro)
@@ -37,5 +37,5 @@
             <origin xyz="0 0 0.4" rpy="0 0 0"/>
             <axis xyz="0 0 1"/>
-            <limit effort="20" velocity="2.0" lower="-3.2" upper="3.2"/>
+            <limit effort="20" velocity="2.0" lower="-6.4" upper="6.4"/>
             <dynamics damping="0.1" friction="0.05"/>
         </joint>
@@ -70,5 +70,5 @@
             <origin xyz="0 -1.0 0.1" rpy="0 0 0"/>
             <axis xyz="0 0 1"/>
-            <limit effort="15" velocity="2.0" lower="-3.2" upper="3.2"/>
+            <limit effort="15" velocity="2.0" lower="-6.4" upper="6.4"/>
             <dynamics damping="0.1" friction="0.05"/>
         </joint>
@@ -134,5 +134,5 @@
             <parent link="gripper_link"/>
             <child link="finger1"/>
-            <origin xyz="0 -0.04 -0.23" rpy="0 0 0"/>
+            <origin xyz="0 -0.04 -0.22" rpy="0 0 0"/>
             <axis xyz="0 1 0"/>
             <limit effort="20" velocity="0.05" lower="0.0" upper="0.04"/>
@@ -143,11 +143,11 @@
                 <origin xyz="0 0 0" rpy="0 0 0"/>
                 <geometry>
-                    <box size="0.02 0.01 0.02"/>
-                </geometry>
-            </collision>
-            <visual>
-                <origin xyz="0 0 0" rpy="0 0 0"/>
-                <geometry>
-                    <box size="0.02 0.01 0.02"/>
+                    <box size="0.03 0.01 0.03"/>
+                </geometry>
+            </collision>
+            <visual>
+                <origin xyz="0 0 0" rpy="0 0 0"/>
+                <geometry>
+                    <box size="0.03 0.01 0.03"/>
                 </geometry>
                 <material name="dark_gray">
@@ -173,5 +173,5 @@
             <parent link="gripper_link"/>
             <child link="finger2"/>
-            <origin xyz="0.04 0 -0.23" rpy="0 0 0"/>
+            <origin xyz="0.04 0 -0.22" rpy="0 0 0"/>
             <axis xyz="1 0 0"/>
             <limit effort="20" velocity="0.05" lower="-0.04" upper="0.0"/>
@@ -182,11 +182,11 @@
                 <origin xyz="0 0 0" rpy="0 0 0"/>
                 <geometry>
-                    <box size="0.01 0.02 0.02"/>
-                </geometry>
-            </collision>
-            <visual>
-                <origin xyz="0 0 0" rpy="0 0 0"/>
-                <geometry>
-                    <box size="0.01 0.02 0.02"/>
+                    <box size="0.01 0.03 0.03"/>
+                </geometry>
+            </collision>
+            <visual>
+                <origin xyz="0 0 0" rpy="0 0 0"/>
+                <geometry>
+                    <box size="0.01 0.03 0.03"/>
                 </geometry>
                 <material name="dark_gray">
@@ -212,5 +212,5 @@
             <parent link="gripper_link"/>
             <child link="finger3"/>
-            <origin xyz="0 0.04 -0.23" rpy="0 0 0"/>
+            <origin xyz="0 0.04 -0.22" rpy="0 0 0"/>
             <axis xyz="0 1 0"/>
             <limit effort="20" velocity="0.05" lower="-0.04" upper="0.0"/>
@@ -221,11 +221,11 @@
                 <origin xyz="0 0 0" rpy="0 0 0"/>
                 <geometry>
-                    <box size="0.02 0.01 0.02"/>
-                </geometry>
-            </collision>
-            <visual>
-                <origin xyz="0 0 0" rpy="0 0 0"/>
-                <geometry>
-                    <box size="0.02 0.01 0.02"/>
+                    <box size="0.03 0.01 0.03"/>
+                </geometry>
+            </collision>
+            <visual>
+                <origin xyz="0 0 0" rpy="0 0 0"/>
+                <geometry>
+                    <box size="0.03 0.01 0.03"/>
                 </geometry>
                 <material name="dark_gray">
@@ -251,5 +251,5 @@
             <parent link="gripper_link"/>
             <child link="finger4"/>
-            <origin xyz="-0.04 0 -0.23" rpy="0 0 0"/>
+            <origin xyz="-0.04 0 -0.22" rpy="0 0 0"/>
             <axis xyz="1 0 0"/>
             <limit effort="20" velocity="0.05" lower="0.0" upper="0.04"/>
@@ -260,11 +260,11 @@
                 <origin xyz="0 0 0" rpy="0 0 0"/>
                 <geometry>
-                    <box size="0.01 0.02 0.02"/>
-                </geometry>
-            </collision>
-            <visual>
-                <origin xyz="0 0 0" rpy="0 0 0"/>
-                <geometry>
-                    <box size="0.01 0.02 0.02"/>
+                    <box size="0.01 0.03 0.03"/>
+                </geometry>
+            </collision>
+            <visual>
+                <origin xyz="0 0 0" rpy="0 0 0"/>
+                <geometry>
+                    <box size="0.01 0.03 0.03"/>
                 </geometry>
                 <material name="dark_gray">

File: src/arm_description/urdf/robot.ros_control.xacro (robot description, xacro)
@@ -83,5 +83,4 @@
                     <arm_name>scara_arm</arm_name>
                     <palm_link>gripper_link</palm_link>
-                    <!-- 注意: finger链路实际名称为 finger1/finger2/finger3/finger4 -->
                     <gripper_link>finger1</gripper_link>
                     <gripper_link>finger2</gripper_link>
@@ -89,5 +88,5 @@
                     <gripper_link>finger4</gripper_link>
                 </arm>
-                <forces_angle_tolerance>100</forces_angle_tolerance>
+                <forces_angle_tolerance>92</forces_angle_tolerance>
                 <update_rate>90</update_rate>
                 <grip_count_threshold>8</grip_count_threshold>

Commit message: [feat]:添加上旋转关节，并成功实现旋转

File: src/arm_description/urdf/base.urdf.xacro (robot description, xacro)
@@ -131,8 +131,42 @@
             <material>Gazebo/White</material>
         </gazebo>
+        <!-- Roll joint for end-effector orientation about Z -->
+        <joint name="gripper_roll" type="revolute">
+            <parent link="gripper_link"/>
+            <child link="gripper_roll_link"/>
+            <origin xyz="0 0 -0.2" rpy="0 0 0"/>
+            <axis xyz="0 0 1"/>
+            <limit effort="10" velocity="3.0" lower="-3.14" upper="3.14"/>
+            <dynamics damping="0.05" friction="0.02"/>
+        </joint>
+        <link name="gripper_roll_link">
+            <collision>
+                <origin xyz="0 0 0" rpy="0 0 0"/>
+                <geometry>
+                    <cylinder length="0.01" radius="0.02"/>
+                </geometry>
+            </collision>
+            <visual>
+                <origin xyz="0 0 0" rpy="0 0 0"/>
+                <geometry>
+                    <cylinder length="0.01" radius="0.02"/>
+                </geometry>
+                <material name="dark">
+                    <color rgba="0.0 0.0 0.0 1.0"/>
+                </material>
+            </visual>
+            <inertial>
+                <origin xyz="0 0 0" rpy="0 0 0"/>
+                <mass value="0.05"/>
+                <inertia ixx="1e-4" ixy="0.0" ixz="0.0" iyy="1e-4" iyz="0.0" izz="1e-4"/>
+            </inertial>
+        </link>
+        <gazebo reference="gripper_roll_link">
+            <material>Gazebo/Dark</material>
+        </gazebo>
         <joint name="finger1_joint" type="prismatic">
-            <parent link="gripper_link"/>
+            <parent link="gripper_roll_link"/>
             <child link="finger1"/>
-            <origin xyz="0 -0.04 -0.22" rpy="0 0 0"/>
+            <origin xyz="0 -0.04 -0.02" rpy="0 0 0"/>
             <axis xyz="0 1 0"/>
             <limit effort="20" velocity="0.05" lower="0.0" upper="0.04"/>
@@ -171,7 +205,7 @@
         </gazebo>
         <joint name="finger2_joint" type="prismatic">
-            <parent link="gripper_link"/>
+            <parent link="gripper_roll_link"/>
             <child link="finger2"/>
-            <origin xyz="0.04 0 -0.22" rpy="0 0 0"/>
+            <origin xyz="0.04 0 -0.02" rpy="0 0 0"/>
             <axis xyz="1 0 0"/>
             <limit effort="20" velocity="0.05" lower="-0.04" upper="0.0"/>
@@ -210,7 +244,7 @@
         </gazebo>
         <joint name="finger3_joint" type="prismatic">
-            <parent link="gripper_link"/>
+            <parent link="gripper_roll_link"/>
             <child link="finger3"/>
-            <origin xyz="0 0.04 -0.22" rpy="0 0 0"/>
+            <origin xyz="0 0.04 -0.02" rpy="0 0 0"/>
             <axis xyz="0 1 0"/>
             <limit effort="20" velocity="0.05" lower="-0.04" upper="0.0"/>
@@ -249,7 +283,7 @@
         </gazebo>
         <joint name="finger4_joint" type="prismatic">
-            <parent link="gripper_link"/>
+            <parent link="gripper_roll_link"/>
             <child link="finger4"/>
-            <origin xyz="-0.04 0 -0.22" rpy="0 0 0"/>
+            <origin xyz="-0.04 0 -0.02" rpy="0 0 0"/>
             <axis xyz="1 0 0"/>
             <limit effort="20" velocity="0.05" lower="0.0" upper="0.04"/>

File: src/arm_description/urdf/robot.ros_control.xacro (robot description, xacro)
@@ -30,4 +30,14 @@
             </joint>
             <actuator name="gripper_motor">
+                <hardwareInterface>hardware_interface/PositionJointInterface</hardwareInterface>
+                <mechanicalReduction>1</mechanicalReduction>
+            </actuator>
+        </transmission>
+        <transmission name="gripper_roll_transmission">
+            <type>transmission_interface/SimpleTransmission</type>
+            <joint name="gripper_roll">
+                <hardwareInterface>hardware_interface/PositionJointInterface</hardwareInterface>
+            </joint>
+            <actuator name="gripper_roll_motor">
                 <hardwareInterface>hardware_interface/PositionJointInterface</hardwareInterface>
                 <mechanicalReduction>1</mechanicalReduction>

Commit message: [feat]:实现下降前对齐，完美解决夹棱角问题

File: src/arm_description/urdf/base.urdf.xacro (robot description, xacro)
@@ -177,11 +177,11 @@
                 <origin xyz="0 0 0" rpy="0 0 0"/>
                 <geometry>
-                    <box size="0.03 0.01 0.03"/>
-                </geometry>
-            </collision>
-            <visual>
-                <origin xyz="0 0 0" rpy="0 0 0"/>
-                <geometry>
-                    <box size="0.03 0.01 0.03"/>
+                    <box size="0.02 0.01 0.02"/>
+                </geometry>
+            </collision>
+            <visual>
+                <origin xyz="0 0 0" rpy="0 0 0"/>
+                <geometry>
+                    <box size="0.02 0.01 0.02"/>
                 </geometry>
                 <material name="dark_gray">
@@ -216,11 +216,11 @@
                 <origin xyz="0 0 0" rpy="0 0 0"/>
                 <geometry>
-                    <box size="0.01 0.03 0.03"/>
-                </geometry>
-            </collision>
-            <visual>
-                <origin xyz="0 0 0" rpy="0 0 0"/>
-                <geometry>
-                    <box size="0.01 0.03 0.03"/>
+                    <box size="0.01 0.02 0.02"/>
+                </geometry>
+            </collision>
+            <visual>
+                <origin xyz="0 0 0" rpy="0 0 0"/>
+                <geometry>
+                    <box size="0.01 0.02 0.02"/>
                 </geometry>
                 <material name="dark_gray">
@@ -255,11 +255,11 @@
                 <origin xyz="0 0 0" rpy="0 0 0"/>
                 <geometry>
-                    <box size="0.03 0.01 0.03"/>
-                </geometry>
-            </collision>
-            <visual>
-                <origin xyz="0 0 0" rpy="0 0 0"/>
-                <geometry>
-                    <box size="0.03 0.01 0.03"/>
+                    <box size="0.02 0.01 0.02"/>
+                </geometry>
+            </collision>
+            <visual>
+                <origin xyz="0 0 0" rpy="0 0 0"/>
+                <geometry>
+                    <box size="0.02 0.01 0.02"/>
                 </geometry>
                 <material name="dark_gray">
@@ -294,11 +294,11 @@
                 <origin xyz="0 0 0" rpy="0 0 0"/>
                 <geometry>
-                    <box size="0.01 0.03 0.03"/>
-                </geometry>
-            </collision>
-            <visual>
-                <origin xyz="0 0 0" rpy="0 0 0"/>
-                <geometry>
-                    <box size="0.01 0.03 0.03"/>
+                    <box size="0.01 0.02 0.02"/>
+                </geometry>
+            </collision>
+            <visual>
+                <origin xyz="0 0 0" rpy="0 0 0"/>
+                <geometry>
+                    <box size="0.01 0.02 0.02"/>
                 </geometry>
                 <material name="dark_gray">
