Commit message: [feat]:实现从世界坐标-相机坐标-图像坐标-像素坐标的正向运动推算

File: src/arm_description/urdf/camera_d435i.urdf.xacro (robot description, xacro)
@@ -40,10 +40,11 @@
             <parent link="camera_link"/>
             <child link="camera_color_optical_frame"/>
-            <origin xyz="0 0 0" rpy="-1.5708 0 -1.5708"/>
+            <!-- Rotate so optical frame aligns with REP-103 when camera_link x:forward, y:right, z:down -->
+            <origin xyz="0 0 0" rpy="1.5708 0 1.5708"/>
         </joint>
         <joint name="camera_depth_optical_joint" type="fixed">
             <parent link="camera_link"/>
             <child link="camera_depth_optical_frame"/>
-            <origin xyz="0 0 0" rpy="-1.5708 0 -1.5708"/>
+            <origin xyz="0 0 0" rpy="1.5708 0 1.5708"/>
         </joint>
         <!-- Gazebo 插件配置：模拟 RealSense D435i -->

Commit message: [feat]:加入yolo，但目前目标太小了，识别不出来，在考虑提升相机参数

File: src/arm_description/urdf/camera_d435i.urdf.xacro (robot description, xacro)
@@ -34,5 +34,5 @@
             <child link="camera_link"/>
             <!-- 放在世界上方，斜135度俯视工作区 -->
-            <origin xyz="3.0 0 2.0" rpy="0 2.356 0"/>
+            <origin xyz="2.0 0 1.5" rpy="0 2.356 0"/>
         </joint>
         <!-- 光学 frame 相对于相机的关节 -->

Commit message: [feat]:调整相机位置，目前方块在图像中大概为12x12，后续如果模型训练不成功的话考虑把机械臂长度减半

File: src/arm_description/urdf/camera_d435i.urdf.xacro (robot description, xacro)
@@ -34,5 +34,5 @@
             <child link="camera_link"/>
             <!-- 放在世界上方，斜135度俯视工作区 -->
-            <origin xyz="2.0 0 1.5" rpy="0 2.356 0"/>
+            <origin xyz="2.8 0 1.65" rpy="0 2.356 0"/>
         </joint>
         <!-- 光学 frame 相对于相机的关节 -->
@@ -52,13 +52,13 @@
             <sensor name="color_camera" type="camera">
                 <camera>
-                    <horizontal_fov>1.047</horizontal_fov>  <!-- 60 度 -->
+                    <horizontal_fov>1.204</horizontal_fov>  <!-- ~69 度，D435i 彩色 FOV -->
                     <image>
-                        <width>640</width>
+                        <width>848</width>
                         <height>480</height>
                         <format>R8G8B8</format>
                     </image>
                     <clip>
-                        <near>0.05</near>
-                        <far>8.0</far>
+                        <near>0.1</near>
+                        <far>6.0</far>
                     </clip>
                 </camera>
@@ -80,12 +80,12 @@
             <sensor name="depth_camera" type="depth">
                 <camera>
-                    <horizontal_fov>1.047</horizontal_fov>
+                    <horizontal_fov>1.518</horizontal_fov> <!-- ~87 度，D435i 深度 FOV -->
                     <image>
-                        <width>640</width>
+                        <width>848</width>
                         <height>480</height>
                     </image>
                     <clip>
-                        <near>0.05</near>
-                        <far>8.0</far>
+                        <near>0.1</near>
+                        <far>6.0</far>
                     </clip>
                 </camera>

Commit message: [feat]:改变相机位置，使方块在图像中占比能到15x15

File: src/arm_description/urdf/camera_d435i.urdf.xacro (robot description, xacro)
@@ -34,5 +34,6 @@
             <child link="camera_link"/>
             <!-- 放在世界上方，斜135度俯视工作区 -->
-            <origin xyz="2.8 0 1.65" rpy="0 2.356 0"/>
+            <!-- <origin xyz="2.8 0 1.65" rpy="0 2.356 0"/> -->
+            <origin xyz="0.5 0 1.3" rpy="0 1.5708 0"/>
         </joint>
         <!-- 光学 frame 相对于相机的关节 -->
