Commit message: [feat]:更新readme，在夹爪下方添加了一个相机；并且发现在gazebo中夹爪旋转有时并不会带着方块一起旋转，不知道是加速度的原因还是别的因素；最后会时把一个物体放到另一个物体上面这样的任务失败

File: src/arm_description/urdf/camera_gripper.urdf.xacro (robot description, xacro)
@@ -1,12 +1,12 @@
 <?xml version="1.0"?>
 <robot xmlns:xacro="http://www.ros.org/wiki/xacro">
-    <!-- D435i 深度相机的 ROS 模拟配置 -->
-    <xacro:macro name="d435i_camera">
+    <!-- gripper_roll下方相机的 ROS 模拟配置-->
+    <xacro:macro name="gripper_camera">
         <!-- 相机 link -->
-        <link name="camera_link">
+        <link name="gripper_camera_link">
             <collision>
                 <origin xyz="0 0 0" rpy="0 0 0"/>
                 <geometry>
-                    <box size="0.09 0.025 0.025"/>
+                    <box size="0.001 0.020 0.020"/>
                 </geometry>
             </collision>
@@ -14,5 +14,5 @@
                 <origin xyz="0 0 0" rpy="0 0 0"/>
                 <geometry>
-                    <box size="0.09 0.025 0.025"/>
+                    <box size="0.001 0.020 0.020"/>
                 </geometry>
                 <material name="dark_gray">
@@ -22,32 +22,32 @@
             <inertial>
                 <origin xyz="0 0 0" rpy="0 0 0"/>
-                <mass value="0.1"/>
-                <inertia ixx="1e-5" ixy="0.0" ixz="0.0" iyy="1e-5" iyz="0.0" izz="1e-5"/>
+                <mass value="0.01"/>
+                <inertia ixx="6.67e-6" ixy="0.0" ixz="0.0" iyy="3.34e-6" iyz="0.0" izz="3.34e-6"/>
             </inertial>
         </link>
         <!-- 光学相机中心 link -->
-        <link name="camera_color_optical_frame"/>
-        <link name="camera_depth_optical_frame"/>
-        <!-- 相机相对于世界的固定关节（俯视） -->
-        <joint name="camera_fixed_joint" type="fixed">
-            <parent link="world"/>
-            <child link="camera_link"/>
+        <link name="gripper_camera_color_optical_frame"/>
+        <link name="gripper_camera_depth_optical_frame"/>
+        <!-- 相机相对于gripper_roll_link的固定关节（俯视） -->
+        <joint name="gripper_camera_fixed_joint" type="fixed">
+            <parent link="gripper_roll_link"/>
+            <child link="gripper_camera_link"/>
             <!-- <origin xyz="2.8 0 1.65" rpy="0 2.356 0"/> -->
-            <origin xyz="0.5 0 1.3" rpy="0 1.5708 0"/>
+            <origin xyz="0.0 0.0 -0.005" rpy="0 1.5708 0"/>
         </joint>
         <!-- 光学 frame 相对于相机的关节 -->
-        <joint name="camera_color_optical_joint" type="fixed">
-            <parent link="camera_link"/>
-            <child link="camera_color_optical_frame"/>
+        <joint name="gripper_camera_color_optical_joint" type="fixed">
+            <parent link="gripper_camera_link"/>
+            <child link="gripper_camera_color_optical_frame"/>
             <!-- Rotate so optical frame aligns with REP-103 when camera_link x:forward, y:right, z:down -->
-            <origin xyz="0 0 0" rpy="1.5708 0 1.5708"/>
+            <origin xyz="0 0 0" rpy="0.0 0.0 0.0"/>
         </joint>
-        <joint name="camera_depth_optical_joint" type="fixed">
-            <parent link="camera_link"/>
-            <child link="camera_depth_optical_frame"/>
-            <origin xyz="0 0 0" rpy="1.5708 0 1.5708"/>
+        <joint name="gripper_camera_depth_optical_joint" type="fixed">
+            <parent link="gripper_camera_link"/>
+            <child link="gripper_camera_depth_optical_frame"/>
+            <origin xyz="0 0 0" rpy="0.0 0 0.0"/>
         </joint>
         <!-- Gazebo 插件配置：模拟 RealSense D435i -->
-        <gazebo reference="camera_link">
+        <gazebo reference="gripper_camera_link">
             <sensor name="color_camera" type="camera">
                 <camera>
@@ -72,13 +72,13 @@
                     <alwaysOn>true</alwaysOn>
                     <updateRate>30.0</updateRate>
-                    <cameraName>camera/color</cameraName>
+                    <cameraName>gripper_camera/color</cameraName>
                     <imageTopicName>image_raw</imageTopicName>
-                    <cameraInfoTopicName>camera_info</cameraInfoTopicName>
-                    <frameName>camera_color_optical_frame</frameName>
+                    <cameraInfoTopicName>gripper_camera_info</cameraInfoTopicName>
+                    <frameName>gripper_camera_color_optical_frame</frameName>
                     <hackBaseline>0.07</hackBaseline>
                 </plugin>
             </sensor>
         </gazebo>
-        <gazebo reference="camera_link">
+        <gazebo reference="gripper_camera_link">
             <sensor name="depth_camera" type="depth">
                 <camera>
@@ -99,11 +99,11 @@
                     <alwaysOn>true</alwaysOn>
                     <updateRate>30.0</updateRate>
-                    <cameraName>camera/depth</cameraName>
+                    <cameraName>gripper_camera/depth</cameraName>
                     <depthImageTopicName>image_rect_raw</depthImageTopicName>
-                    <cameraInfoTopicName>camera_info</cameraInfoTopicName>
-                    <pointCloudTopicName>points</pointCloudTopicName>
+                    <cameraInfoTopicName>gripper_camera_info</cameraInfoTopicName>
+                    <pointCloudTopicName>gripper_points</pointCloudTopicName>
                     <pointCloudCutoff>0.05</pointCloudCutoff>
                     <pointCloudCutoffMax>8.0</pointCloudCutoffMax>
-                    <frameName>camera_depth_optical_frame</frameName>
+                    <frameName>gripper_camera_depth_optical_frame</frameName>
                 </plugin>
             </sensor>

File: src/arm_description/urdf/scara.urdf.xacro (robot description, xacro)
@@ -4,6 +4,8 @@
     <xacro:include filename="$(find arm_description)/urdf/robot.ros_control.xacro"/>
     <xacro:include filename="$(find arm_description)/urdf/camera_d435i.urdf.xacro"/>
+    <xacro:include filename="$(find arm_description)/urdf/camera_gripper.urdf.xacro"/>
     <xacro:base_xacro/>
     <xacro:robot_ros_control/>
     <xacro:d435i_camera/>
+    <xacro:gripper_camera/>
 </robot>

Commit message: [feat]:加入gripper相机相关的处理节点，已经可以可视化拍到的画面，下一步是加入深度处理逻辑

File: src/arm_description/urdf/camera_gripper.urdf.xacro (robot description, xacro)
@@ -41,10 +41,10 @@
             <child link="gripper_camera_color_optical_frame"/>
             <!-- Rotate so optical frame aligns with REP-103 when camera_link x:forward, y:right, z:down -->
-            <origin xyz="0 0 0" rpy="0.0 0.0 0.0"/>
+            <origin xyz="0 0 0" rpy="1.5708 0 1.5708"/>
         </joint>
         <joint name="gripper_camera_depth_optical_joint" type="fixed">
             <parent link="gripper_camera_link"/>
             <child link="gripper_camera_depth_optical_frame"/>
-            <origin xyz="0 0 0" rpy="0.0 0 0.0"/>
+            <origin xyz="0 0 0" rpy="1.5708 0 1.5708"/>
         </joint>
         <!-- Gazebo 插件配置：模拟 RealSense D435i -->
