Commit message: [feat]:修改全局摄像机位置，让视角更合理

File: src/arm_description/urdf/world_camera.urdf.xacro (robot description, xacro)
@@ -33,5 +33,5 @@
             <child link="world_camera_link"/>
             <!-- 推荐观察位姿 -->
-            <origin xyz="1.6 -1.5 1.0" rpy="0 0.75 2.35"/>
+            <origin xyz="2.0 -1.5 1.0" rpy="0 0.5236 2.618"/>
         </joint>
         <!-- optical frame -->
